Commit message: fix bounds for joint

File: pr2_examples_gazebo/single_link_defs/single_link.transmission.xacro (robot description, xacro)
@@ -6,5 +6,4 @@
     <mechanicalReduction>1</mechanicalReduction>
     <motorTorqueConstant>1</motorTorqueConstant>
-    <pulsesPerRevolution>90000</pulsesPerRevolution>
   </transmission>
 </robot>

File: pr2_examples_gazebo/single_link_defs/single_link.urdf.xacro (robot description, xacro)
@@ -42,5 +42,5 @@
   <joint name="link1_joint" type="revolute" >
     <axis xyz="1 0 0" />
-    <limit upper="-3" lower="3" effort="100" velocity="5" />
+    <limit upper="1" lower="-1" effort="100" velocity="5" />
     <parent link="base_block" />
     <origin xyz="0 0 1" rpy="0 0 0" />
