Commit message: update single link

File: pr2_examples_gazebo/single_link_defs/single_link.urdf.xacro (robot description, xacro)
@@ -42,5 +42,5 @@
   <joint name="link1_joint" type="revolute" >
     <axis xyz="1 0 0" />
-    <limit upper="1" lower="-1" effort="100" velocity="5" />
+    <limit upper="2" lower="-2" effort="100" velocity="5" />
     <parent link="base_block" />
     <origin xyz="0 0 1" rpy="0 0 0" />
@@ -73,5 +73,5 @@
       <controller:gazebo_ros_time name="gazebo_ros_time" plugin="libgazebo_ros_time.so">
         <alwaysOn>true</alwaysOn>
-        <updateRate>100.0</updateRate>
+        <updateRate>1000.0</updateRate>
         <interface:audio name="dummy_gazebo_ros_time_iface_should_not_be_here"/>
       </controller:gazebo_ros_time>
@@ -79,5 +79,5 @@
       <controller:gazebo_ros_controller_manager name="gazebo_ros_controller_manager" plugin="libgazebo_ros_controller_manager.so">
         <alwaysOn>true</alwaysOn>
-        <updateRate>100.0</updateRate>
+        <updateRate>1000.0</updateRate>
         <interface:audio name="gazebo_ros_controller_manager_dummy_iface" />
       </controller:gazebo_ros_controller_manager>
@@ -85,5 +85,5 @@
       <controller:gazebo_ros_p3d name="p3d_link1_controller" plugin="libgazebo_ros_p3d.so">
           <alwaysOn>true</alwaysOn>
-          <updateRate>100.0</updateRate>
+          <updateRate>1000.0</updateRate>
           <bodyName>link1</bodyName>
           <topicName>link1_pose</topicName>
