Commit message: updates for #3036.

File: pr2_examples_gazebo/dual_link_defs/dual_link.urdf.xacro (robot description, xacro)
@@ -15,5 +15,5 @@
   <joint name="base_block_joint" type="fixed">
     <parent link="world" />
-    <origin xyz="0 0 0.002 " rpy="0 0 0" />
+    <origin xyz="0 0 0" rpy="0 0 0" />
     <child link="base_block" />
   </joint>
@@ -41,26 +41,26 @@
   </gazebo>
   <joint name="link1_joint" type="revolute" >
-    <axis xyz="1 0 0" />
-    <limit upper="-3.14159" lower="3.14159" effort="100" velocity="5" />
+    <axis xyz="0 0 1" />
+    <limit lower="0.0" upper="0.0" effort="100" velocity="5" />
     <parent link="base_block" />
-    <origin xyz="0 0 1" rpy="0 0 0" />
+    <origin xyz="0 0 2" rpy="0 0 0" />
     <child link="link1" />
   </joint>
   <link name="link1">
     <inertial >
-      <mass value="10" />
-      <origin xyz="0 0 0" />
-      <inertia  ixx="1.0" ixy="0.0"  ixz="0.0"  iyy="0.1"  iyz="0.0"  izz="0.1" />
+      <mass value="0.1" />
+      <origin xyz="0 0 -0.5" />
+      <inertia  ixx="0.1" ixy="0.0"  ixz="0.0"  iyy="0.1"  iyz="0.0"  izz="0.1" />
     </inertial>
     <visual >
-      <origin xyz="0 0 0" rpy="0 0 0" />
-      <geometry name="sholder_roll_mesh_file">
-        <box size="1.0 0.3 0.3" />
+      <origin xyz="0 0 -0.5" rpy="0 0 0" />
+      <geometry name="link1_visual_geom">
+        <box size="0.1 0.1 1.0" />
       </geometry>
     </visual>
     <collision >
-      <origin xyz="0.5 0 0" rpy="0.0 0.0 0.0 " />
+      <origin xyz="0 0 -0.5" rpy="0.0 0.0 0.0 " />
       <geometry name="link1_collision_geom">
-        <box size="1.0 0.3 0.3" />
+        <box size="0.1 0.1 1.0" />
       </geometry>
     </collision>
@@ -68,31 +68,71 @@
   <gazebo reference="link1">
     <material>Gazebo/Red</material>
-    <turnGravityOff>true</turnGravityOff>
+    <turnGravityOff>false</turnGravityOff>
   </gazebo>
+  <joint name="link2_joint" type="continuous" >
+    <axis xyz="0 1 0" />
+    <limit effort="100" velocity="5" />
+    <dynamics damping="0.0" friction="0.0" />
+    <parent link="link1" />
+    <origin xyz="0 0 0" rpy="0 90 0" />
+    <child link="link2" />
+  </joint>
+  <link name="link2">
+    <inertial >
+      <mass value="1.0" />
+      <origin xyz="0 0 0.5" />
+      <inertia  ixx="1.0" ixy="0.0"  ixz="0.0"  iyy="1.0"  iyz="0.0"  izz="1.0" />
+    </inertial>
+    <visual >
+      <origin xyz="0 0 0.5" rpy="0 0 0" />
+      <geometry name="link2_visual_geom">
+        <cylinder radius="0.05" length="1.0" />
+      </geometry>
+    </visual>
+    <collision >
+      <origin xyz="0 0 0.5" rpy="0 0 0 " />
+      <geometry name="link2_collision_geom">
+        <cylinder radius="0.05" length="1.0" />
+      </geometry>
+    </collision>
+  </link>
+  <gazebo reference="link2">
+    <material>Gazebo/Blue</material>
+    <turnGravityOff>false</turnGravityOff>
+  </gazebo>
+  <!-- mechanism controls -->
+  <include filename="./dual_link.transmission.xacro" />
   <gazebo>
       <controller:ros_time name="ros_time" plugin="libros_time.so">
         <alwaysOn>true</alwaysOn>
-        <updateRate>100.0</updateRate>
+        <updateRate>1000.0</updateRate>
         <interface:audio name="dummy_ros_time_iface_should_not_be_here"/>
       </controller:ros_time>
-      <!-- PR2_ACTARRAY -->
-      <controller:gazebo_controller_manager name="gazebo_controller_manager" plugin="libgazebo_controller_manager.so">
+      <!-- pr2_actarray -->
+      <controller:ros_controller_manager name="ros_controller_manager" plugin="libros_controller_manager.so">
         <alwaysOn>true</alwaysOn>
-        <updateRate>100.0</updateRate>
-        <interface:audio name="gazebo_controller_manager_dummy_iface" />
-      </controller:gazebo_controller_manager>
+        <updateRate>1000.0</updateRate>
+        <interface:audio name="ros_controller_manager_dummy_iface" />
+      </controller:ros_controller_manager>
       <!-- ros_p3d for position groundtruth -->
       <controller:ros_p3d name="p3d_link1_controller" plugin="libros_p3d.so">
           <alwaysOn>true</alwaysOn>
-          <updateRate>100.0</updateRate>
+          <updateRate>1000.0</updateRate>
           <bodyName>link1</bodyName>
           <topicName>link1_pose</topicName>
           <frameName>map</frameName>
+          <xyzOffsets>0 0 0.0</xyzOffsets>
+          <rpyOffsets>0 0 0.0</rpyOffsets>
           <interface:position name="p3d_link1_position"/>
       </controller:ros_p3d>
+      <!-- ros_p3d for position groundtruth -->
+      <controller:ros_p3d name="p3d_link2_controller" plugin="libros_p3d.so">
+          <alwaysOn>true</alwaysOn>
+          <updateRate>1000.0</updateRate>
+          <bodyName>link2</bodyName>
+          <topicName>link2_pose</topicName>
+          <frameName>map</frameName>
+          <interface:position name="p3d_link2_position"/>
+      </controller:ros_p3d>
   </gazebo>
-  <!-- Define groups of links; a link may be part of multiple groups -->
-  <include filename="./groups_single_link.xml" />
-  <!-- mechanism controls -->
-  <include filename="./transmissions_single_link.xml" />
 </robot>

File: pr2_examples_gazebo/multi_link_defs/multi_link.urdf.xacro (robot description, xacro)
@@ -272,8 +272,6 @@
     <turnGravityOff>false</turnGravityOff>
   </gazebo>
-  <!-- Define groups of links; a link may be part of multiple groups -->
-  <include filename="./groups_multi_link.xml" />
   <!-- mechanism controls -->
-  <include filename="./transmissions_multi_link.xml" />
+  <include filename="./multi_link.transmission.xacro" />
   <gazebo>
       <controller:ros_time name="ros_time" plugin="libros_time.so">
@@ -283,9 +281,9 @@
       </controller:ros_time>
       <!-- PR2_ACTARRAY -->
-      <controller:gazebo_controller_manager name="gazebo_controller_manager" plugin="libgazebo_controller_manager.so">
+      <controller:ros_controller_manager name="ros_controller_manager" plugin="libros_controller_manager.so">
         <alwaysOn>true</alwaysOn>
         <updateRate>1000.0</updateRate>
-        <interface:audio name="gazebo_controller_manager_dummy_iface" />
-      </controller:gazebo_controller_manager>
+        <interface:audio name="ros_controller_manager_dummy_iface" />
+      </controller:ros_controller_manager>
       <!-- ros_p3d for position groundtruth -->
       <controller:ros_p3d name="p3d_link3_controller" plugin="libros_p3d.so">

File: pr2_examples_gazebo/single_link_defs/single_link.urdf.xacro (robot description, xacro)
@@ -15,5 +15,5 @@
   <joint name="base_block_joint" type="fixed">
     <parent link="world" />
-    <origin xyz="0 0 0" rpy="0 0 0" />
+    <origin xyz="0 0 0.002 " rpy="0 0 0" />
     <child link="base_block" />
   </joint>
@@ -41,26 +41,26 @@
   </gazebo>
   <joint name="link1_joint" type="revolute" >
-    <axis xyz="0 0 1" />
-    <limit lower="0.0" upper="0.0" effort="100" velocity="5" />
+    <axis xyz="1 0 0" />
+    <limit upper="-3" lower="3" effort="100" velocity="5" />
     <parent link="base_block" />
-    <origin xyz="0 0 2" rpy="0 0 0" />
+    <origin xyz="0 0 1" rpy="0 0 0" />
     <child link="link1" />
   </joint>
   <link name="link1">
     <inertial >
-      <mass value="0.1" />
-      <origin xyz="0 0 -0.5" />
-      <inertia  ixx="0.1" ixy="0.0"  ixz="0.0"  iyy="0.1"  iyz="0.0"  izz="0.1" />
+      <mass value="10" />
+      <origin xyz="0 0 0" />
+      <inertia  ixx="1.0" ixy="0.0"  ixz="0.0"  iyy="0.1"  iyz="0.0"  izz="0.1" />
     </inertial>
     <visual >
-      <origin xyz="0 0 -0.5" rpy="0 0 0" />
-      <geometry name="link1_visual_geom">
-        <box size="0.1 0.1 1.0" />
+      <origin xyz="0 0 0" rpy="0 0 0" />
+      <geometry name="sholder_roll_mesh_file">
+        <box size="1.0 0.3 0.3" />
       </geometry>
     </visual>
     <collision >
-      <origin xyz="0 0 -0.5" rpy="0.0 0.0 0.0 " />
+      <origin xyz="0.5 0 0" rpy="0.0 0.0 0.0 " />
       <geometry name="link1_collision_geom">
-        <box size="0.1 0.1 1.0" />
+        <box size="1.0 0.3 0.3" />
       </geometry>
     </collision>
@@ -68,73 +68,29 @@
   <gazebo reference="link1">
     <material>Gazebo/Red</material>
-    <turnGravityOff>false</turnGravityOff>
+    <turnGravityOff>true</turnGravityOff>
   </gazebo>
-  <joint name="link2_joint" type="continuous" >
-    <axis xyz="0 1 0" />
-    <limit effort="100" velocity="5" />
-    <dynamics damping="0.0" friction="0.0" />
-    <parent link="link1" />
-    <origin xyz="0 0 0" rpy="0 90 0" />
-    <child link="link2" />
-  </joint>
-  <link name="link2">
-    <inertial >
-      <mass value="1.0" />
-      <origin xyz="0 0 0.5" />
-      <inertia  ixx="1.0" ixy="0.0"  ixz="0.0"  iyy="1.0"  iyz="0.0"  izz="1.0" />
-    </inertial>
-    <visual >
-      <origin xyz="0 0 0.5" rpy="0 0 0" />
-      <geometry name="link2_visual_geom">
-        <cylinder radius="0.05" length="1.0" />
-      </geometry>
-    </visual>
-    <collision >
-      <origin xyz="0 0 0.5" rpy="0 0 0 " />
-      <geometry name="link2_collision_geom">
-        <cylinder radius="0.05" length="1.0" />
-      </geometry>
-    </collision>
-  </link>
-  <gazebo reference="link2">
-    <material>Gazebo/Blue</material>
-    <turnGravityOff>false</turnGravityOff>
-  </gazebo>
-  <!-- Define groups of links; a link may be part of multiple groups -->
-  <include filename="./groups_dual_link.xml" />
-  <!-- mechanism controls -->
-  <include filename="./transmissions_dual_link.xml" />
   <gazebo>
       <controller:ros_time name="ros_time" plugin="libros_time.so">
         <alwaysOn>true</alwaysOn>
-        <updateRate>1000.0</updateRate>
+        <updateRate>100.0</updateRate>
         <interface:audio name="dummy_ros_time_iface_should_not_be_here"/>
       </controller:ros_time>
-      <!-- pr2_actarray -->
-      <controller:gazebo_controller_manager name="gazebo_controller_manager" plugin="libgazebo_controller_manager.so">
+      <!-- PR2_ACTARRAY -->
+      <controller:ros_controller_manager name="ros_controller_manager" plugin="libros_controller_manager.so">
         <alwaysOn>true</alwaysOn>
-        <updateRate>1000.0</updateRate>
-        <interface:audio name="gazebo_controller_manager_dummy_iface" />
-      </controller:gazebo_controller_manager>
+        <updateRate>100.0</updateRate>
+        <interface:audio name="ros_controller_manager_dummy_iface" />
+      </controller:ros_controller_manager>
       <!-- ros_p3d for position groundtruth -->
       <controller:ros_p3d name="p3d_link1_controller" plugin="libros_p3d.so">
           <alwaysOn>true</alwaysOn>
-          <updateRate>1000.0</updateRate>
+          <updateRate>100.0</updateRate>
           <bodyName>link1</bodyName>
           <topicName>link1_pose</topicName>
           <frameName>map</frameName>
-          <xyzOffsets>0 0 0.0</xyzOffsets>
-          <rpyOffsets>0 0 0.0</rpyOffsets>
           <interface:position name="p3d_link1_position"/>
       </controller:ros_p3d>
-      <!-- ros_p3d for position groundtruth -->
-      <controller:ros_p3d name="p3d_link2_controller" plugin="libros_p3d.so">
-          <alwaysOn>true</alwaysOn>
-          <updateRate>1000.0</updateRate>
-          <bodyName>link2</bodyName>
-          <topicName>link2_pose</topicName>
-          <frameName>map</frameName>
-          <interface:position name="p3d_link2_position"/>
-      </controller:ros_p3d>
   </gazebo>
+  <!-- mechanism controls -->
+  <include filename="./single_link.transmission.xacro" />
 </robot>

Commit message: Fixed a degree/radian problem

File: pr2_examples_gazebo/dual_link_defs/dual_link.urdf.xacro (robot description, xacro)
@@ -75,5 +75,5 @@
     <dynamics damping="0.0" friction="0.0" />
     <parent link="link1" />
-    <origin xyz="0 0 0" rpy="0 90 0" />
+    <origin xyz="0 0 0" rpy="0 1.57 0" />
     <child link="link2" />
   </joint>

Commit message: cleanup urdfs for example links

File: pr2_examples_gazebo/dual_link_defs/dual_link.urdf.xacro (robot description, xacro)
@@ -26,5 +26,5 @@
     <visual>
       <origin xyz="0 0 0" rpy="0 0 0" />
-      <geometry name="base_block_visual_geom">
+      <geometry>
         <box size="0.001 0.001 0.001" />
       </geometry>
@@ -32,5 +32,5 @@
     <collision>
       <origin xyz="0 0 0" rpy="0.0 0.0 0.0" />
-      <geometry name="base_block_collision_geom">
+      <geometry>
         <box size="0.001 0.001 0.001" />
       </geometry>
@@ -55,11 +55,11 @@
     <visual >
       <origin xyz="0 0 -0.5" rpy="0 0 0" />
-      <geometry name="link1_visual_geom">
+      <geometry>
         <box size="0.1 0.1 1.0" />
       </geometry>
     </visual>
     <collision >
-      <origin xyz="0 0 -0.5" rpy="0.0 0.0 0.0 " />
-      <geometry name="link1_collision_geom">
+      <origin xyz="0 0 -0.5" rpy="0.0 0.0 0.0" />
+      <geometry>
         <box size="0.1 0.1 1.0" />
       </geometry>
@@ -86,11 +86,11 @@
     <visual >
       <origin xyz="0 0 0.5" rpy="0 0 0" />
-      <geometry name="link2_visual_geom">
+      <geometry>
         <cylinder radius="0.05" length="1.0" />
       </geometry>
     </visual>
     <collision >
-      <origin xyz="0 0 0.5" rpy="0 0 0 " />
-      <geometry name="link2_collision_geom">
+      <origin xyz="0 0 0.5" rpy="0 0 0" />
+      <geometry>
         <cylinder radius="0.05" length="1.0" />
       </geometry>

File: pr2_examples_gazebo/multi_link_defs/multi_link.urdf.xacro (robot description, xacro)
@@ -16,5 +16,5 @@
   <joint name="base_block_joint" type="fixed" >
     <parent link="world" />
-    <origin xyz="0 0 0.002 " rpy="0 0 0" />
+    <origin xyz="0 0 0.002" rpy="0 0 0" />
     <child link="base_block" />
   </joint>
@@ -27,5 +27,5 @@
     <visual>
       <origin xyz="0 0 0" rpy="0 0 0" />
-      <geometry name="base_block_visual_geom">
+      <geometry>
         <box size="0.001 0.001 0.001" />
       </geometry>
@@ -33,5 +33,5 @@
     <collision>
       <origin xyz="0 0 0" rpy="0.0 0.0 0.0" />
-      <geometry name="base_block_collision_geom">
+      <geometry>
         <box size="0.001 0.001 0.001" />
       </geometry>
@@ -59,11 +59,11 @@
     <visual >
       <origin xyz="0 0 -0.5" rpy="0 0 0" />
-      <geometry name="link1_visual_geom">
+      <geometry>
         <box size="0.1 0.1 1.0" />
       </geometry>
     </visual>
     <collision >
-      <origin xyz="0 0 -0.5" rpy="0.0 0.0 0.0 " />
-      <geometry name="link1_collision_geom">
+      <origin xyz="0 0 -0.5" rpy="0.0 0.0 0.0" />
+      <geometry>
         <box size="0.1 0.1 1.0" />
       </geometry>
@@ -92,11 +92,11 @@
     <visual >
       <origin xyz="0.5 0 0" rpy="0 0 0" />
-      <geometry name="link2_visual_geom">
-        <box size="1.0 0.1 0.1" />
-      </geometry>
-    </visual>
-    <collision >
-      <origin xyz="0.5 0 0" rpy="0.0 0.0 0.0 " />
-      <geometry name="link2_collision_geom">
+      <geometry>
+        <box size="1.0 0.1 0.1" />
+      </geometry>
+    </visual>
+    <collision >
+      <origin xyz="0.5 0 0" rpy="0.0 0.0 0.0" />
+      <geometry>
         <box size="1.0 0.1 0.1" />
       </geometry>
@@ -125,11 +125,11 @@
     <visual >
       <origin xyz="0.5 0 0" rpy="0 0 0" />
-      <geometry name="link3_visual_geom">
-        <box size="1.0 0.1 0.1" />
-      </geometry>
-    </visual>
-    <collision >
-      <origin xyz="0.5 0 0" rpy="0.0 0.0 0.0 " />
-      <geometry name="link3_collision_geom">
+      <geometry>
+        <box size="1.0 0.1 0.1" />
+      </geometry>
+    </visual>
+    <collision >
+      <origin xyz="0.5 0 0" rpy="0.0 0.0 0.0" />
+      <geometry>
         <box size="1.0 0.1 0.1" />
       </geometry>
@@ -158,11 +158,11 @@
     <visual >
       <origin xyz="0.5 0 0" rpy="0 0 0" />
-      <geometry name="link4_visual_geom">
-        <box size="1.0 0.1 0.1" />
-      </geometry>
-    </visual>
-    <collision >
-      <origin xyz="0.5 0 0" rpy="0.0 0.0 0.0 " />
-      <geometry name="link4_collision_geom">
+      <geometry>
+        <box size="1.0 0.1 0.1" />
+      </geometry>
+    </visual>
+    <collision >
+      <origin xyz="0.5 0 0" rpy="0.0 0.0 0.0" />
+      <geometry>
         <box size="1.0 0.1 0.1" />
       </geometry>
@@ -191,11 +191,11 @@
     <visual >
       <origin xyz="0.5 0 0" rpy="0 0 0" />
-      <geometry name="link5_visual_geom">
-        <box size="1.0 0.1 0.1" />
-      </geometry>
-    </visual>
-    <collision >
-      <origin xyz="0.5 0 0" rpy="0.0 0.0 0.0 " />
-      <geometry name="link5_collision_geom">
+      <geometry>
+        <box size="1.0 0.1 0.1" />
+      </geometry>
+    </visual>
+    <collision >
+      <origin xyz="0.5 0 0" rpy="0.0 0.0 0.0" />
+      <geometry>
         <box size="1.0 0.1 0.1" />
       </geometry>
@@ -224,11 +224,11 @@
     <visual >
       <origin xyz="0.5 0 0" rpy="0 0 0" />
-      <geometry name="link6_visual_geom">
-        <box size="1.0 0.1 0.1" />
-      </geometry>
-    </visual>
-    <collision >
-      <origin xyz="0.5 0 0" rpy="0.0 0.0 0.0 " />
-      <geometry name="link6_collision_geom">
+      <geometry>
+        <box size="1.0 0.1 0.1" />
+      </geometry>
+    </visual>
+    <collision >
+      <origin xyz="0.5 0 0" rpy="0.0 0.0 0.0" />
+      <geometry>
         <box size="1.0 0.1 0.1" />
       </geometry>
@@ -257,11 +257,11 @@
     <visual >
       <origin xyz="0.5 0 0" rpy="0 0 0" />
-      <geometry name="link7_visual_geom">
-        <box size="1.0 0.1 0.1" />
-      </geometry>
-    </visual>
-    <collision >
-      <origin xyz="0.5 0 0" rpy="0.0 0.0 0.0 " />
-      <geometry name="link7_collision_geom">
+      <geometry>
+        <box size="1.0 0.1 0.1" />
+      </geometry>
+    </visual>
+    <collision >
+      <origin xyz="0.5 0 0" rpy="0.0 0.0 0.0" />
+      <geometry>
         <box size="1.0 0.1 0.1" />
       </geometry>

File: pr2_examples_gazebo/single_link_defs/single_link.urdf.xacro (robot description, xacro)
@@ -26,5 +26,5 @@
     <visual>
       <origin xyz="0 0 0" rpy="0 0 0" />
-      <geometry name="base_block_visual_geom">
+      <geometry>
         <box size="0.001 0.001 0.001" />
       </geometry>
@@ -32,5 +32,5 @@
     <collision>
       <origin xyz="0 0 0" rpy="0.0 0.0 0.0" />
-      <geometry name="base_block_collision_geom">
+      <geometry>
         <box size="0.001 0.001 0.001" />
       </geometry>
@@ -55,5 +55,5 @@
     <visual >
       <origin xyz="0 0 0" rpy="0 0 0" />
-      <geometry name="sholder_roll_mesh_file">
+      <geometry>
         <box size="1.0 0.3 0.3" />
       </geometry>
@@ -61,5 +61,5 @@
     <collision >
       <origin xyz="0.5 0 0" rpy="0.0 0.0 0.0 " />
-      <geometry name="link1_collision_geom">
+      <geometry>
         <box size="1.0 0.3 0.3" />
       </geometry>

Commit message: world link definition needed for urdf

File: pr2_examples_gazebo/dual_link_defs/dual_link.urdf.xacro (robot description, xacro)
@@ -13,4 +13,5 @@
        xmlns:controller="http://playerstage.sourceforge.net/gazebo/xmlschema/#controller"
        xmlns:physics="http://playerstage.sourceforge.net/gazebo/xmlschema/#physics">
+  <link name="world"/>
   <joint name="base_block_joint" type="fixed">
     <parent link="world" />

File: pr2_examples_gazebo/multi_link_defs/multi_link.urdf.xacro (robot description, xacro)
@@ -14,4 +14,5 @@
        xmlns:physics="http://playerstage.sourceforge.net/gazebo/xmlschema/#physics">
   <!-- joint blocks -->
+  <link name="world"/>
   <joint name="base_block_joint" type="fixed" >
     <parent link="world" />

File: pr2_examples_gazebo/single_link_defs/single_link.urdf.xacro (robot description, xacro)
@@ -13,4 +13,5 @@
        xmlns:controller="http://playerstage.sourceforge.net/gazebo/xmlschema/#controller"
        xmlns:physics="http://playerstage.sourceforge.net/gazebo/xmlschema/#physics">
+  <link name="world"/>
   <joint name="base_block_joint" type="fixed">
     <parent link="world" />
